Commit message: adjustmanents to lane traking and controllers

File: src/my_f1tenth_sim/urdf/car.xacro (robot description, xacro)
@@ -54,5 +54,5 @@
     <visual>
       <geometry><box size="0.02 0.20 0.04"/></geometry>
-      <material name="white"/>
+      <material name="black"/>
     </visual>
   </link>
@@ -78,5 +78,5 @@
         <origin rpy="${pi/2} 0 0"/>
         <geometry><cylinder radius="${wheel_radius}" length="${wheel_width}"/></geometry>
-        <material name="white"/>
+        <material name="black"/>
       </visual>
       <collision>
@@ -180,5 +180,15 @@
        kp=1e7, kd=1, mu=0.7, maxVel=0.01
        Front wheels keep mu2=0.2 for Ackermann lateral slip; rear=0.7 for traction -->
+  <gazebo reference="base_link">
+    <material>Gazebo/Blue</material>
+  </gazebo>
+  <gazebo reference="bumper">
+    <material>Gazebo/Blue</material>
+  </gazebo>
+  <gazebo reference="raspi">
+    <material>Gazebo/Blue</material>
+  </gazebo>
   <gazebo reference="front_left_wheel">
+    <material>Gazebo/Blue</material>
     <mu1>0.7</mu1>
     <mu2>0.2</mu2>
@@ -190,4 +200,5 @@
   </gazebo>
   <gazebo reference="front_right_wheel">
+    <material>Gazebo/Blue</material>
     <mu1>0.7</mu1>
     <mu2>0.2</mu2>
@@ -199,4 +210,5 @@
   </gazebo>
   <gazebo reference="rear_left_wheel">
+    <material>Gazebo/Blue</material>
     <mu1>0.7</mu1>
     <mu2>0.7</mu2>
@@ -208,4 +220,5 @@
   </gazebo>
   <gazebo reference="rear_right_wheel">
+    <material>Gazebo/Blue</material>
     <mu1>0.7</mu1>
     <mu2>0.7</mu2>
@@ -217,4 +230,5 @@
   </gazebo>
   <gazebo reference="camera_link">
+    <material>Gazebo/Blue</material>
     <sensor name="camera" type="camera">
       <update_rate>30</update_rate>
